File: scard/scard.brd (EAGLE design)
At the start: 47 x 86.5 mm, 70 parts, among them P1 TPS548A20, Q1 FDN360P, T1 LT3652, X1 COAX, X2 1365-20

Commit message: better power traces for voltage regulator
Routing:
- net GND: track 160.3 -> 192.5 mm, vias 102 -> 103
- net VSYS_UNREG: track 63.0 -> 71.9 mm
- net N$2: track 14.5 -> 19.4 mm
